File: circuit/control.kicad_sch (KiCad schematic)
At the start: 0 parts

Commit message: update
Parts:
- added U44, U45, U46: AT28C64B, symbol proc:AT28C64B
- added U47, U48, U49, U50: 74HC238, symbol proc:74HC238
- added U51: 4075, symbol 4xxx:4075
- added U52, U53, U54: 74LS32, symbol 74xx:74LS32
- added U? (x7): 74HC04, symbol 74xx:74HC04
Connections:
- new net: U47.11 (Y4), U53.1
- new net: U48.11 (Y4), U53.2
- new net: U50.10 (Y5), U51.4
- new net: U50.11 (Y4), U54.2
- new net: U50.12 (Y3), U53.13
- new net: U50.13 (Y2), U53.10
- new net: U50.14 (Y1), U53.5
- new net: U50.15 (Y0), U51.13
- new net: U45.13 (D2), U50.6 (E3)
- new net: U49.10 (Y5), U51.3
- new net: U49.11 (Y4), U54.1
- new net: U49.12 (Y3), U53.12
- new net: U49.13 (Y2), U53.9
- new net: U49.14 (Y1), U53.4
- new net: U49.15 (Y0), U51.12
- new net: U45.12 (D1), U49.6 (E3)
- new net: U47.15 (Y0), U52.1
- new net: U48.15 (Y0), U52.2
- new net: U48.10 (Y5), U51.8
- new net: U48.12 (Y3), U52.13
- new net: U48.13 (Y2), U52.10
- new net: U48.14 (Y1), U52.5
- new net: U45.11 (D0), U48.6 (E3)
- new net: U44.17 (D5), U51.5
- new net: U47.13 (Y2), U52.9
- new net: U47.12 (Y3), U52.12
- new net: U44.13 (D2), U51.1
- new net: U47.10 (Y5), U51.2
- new net: U45.15 (D3), U51.11
- new net: U44.19 (D7), U47.6 (E3)
- new net: U47.14 (Y1), U52.4
- new net ALU_A_WE: U46.11 (D0)
- new net ALU_B_WE: U46.12 (D1)
- new net ALU_OE: U46.13 (D2)
- new net A_OE: U52.3
- new net A_WE: U51.10
- new net B_OE: U52.6
- new net B_WE: U53.6
- new net C_OE: U52.8
- new net C_WE: U53.8
- new net D_OE: U52.11
- new net D_WE: U53.11
- new net E_OE: U53.3
- new net E_WE: U54.3
- new net GND: U44.14 (GND), U44.2 (A12), U44.20 (~{CE}), U44.21 (A10), U44.22 (~{OE}), U44.23 (A11), U44.24 (A9), U44.25 (A8), U44.3 (A7), U45.14 (GND), U45.2 (A12), U45.20 (~{CE}), U45.21 (A10), U45.22 (~{OE}), U45.23 (A11), U45.24 (A9), U45.25 (A8), U45.3 (A7), U46.14 (GND), U46.2 (A12), U46.20 (~{CE}), U46.21 (A10), U46.22 (~{OE}), U46.23 (A11), U46.24 (A9), U46.25 (A8), U46.3 (A7), U47.4 (~{E1}), U47.5 (~{E2}), U47.8 (GND), U48.4 (~{E1}), U48.5 (~{E2}), U48.8 (GND), U49.4 (~{E1}), U49.5 (~{E2}), U49.8 (GND), U50.4 (~{E1}), U50.5 (~{E2}), U50.8 (GND), U51.7 (VSS), U52.7 (GND), U53.7 (GND), U54.7 (GND)
- new net HLT: U46.15 (D3)
- new net I0: U44.7 (A3), U45.7 (A3), U46.7 (A3)
- new net I1: U44.6 (A4), U45.6 (A4), U46.6 (A4)
- new net I10: U47.3 (A2), U49.3 (A2)
- new net I12: U48.1 (A0), U50.1 (A0)
- new net I13: U48.2 (A1), U50.2 (A1)
- new net I14: U48.3 (A2), U50.3 (A2)
- new net I2: U44.5 (A5), U45.5 (A5), U46.5 (A5)
- new net I3: U44.4 (A6), U45.4 (A6), U46.4 (A6)
- new net I8: U47.1 (A0), U49.1 (A0)
- new net I9: U47.2 (A1), U49.2 (A1)
- new net IR_WE: U44.18 (D6)
- new net MAR2RAM: U44.11 (D0)
- new net MAR_WE: U44.16 (D4)
- new net MDR_DB: U45.16 (D4)
- new net MDR_OE: U44.12 (D1)
- new net MDR_WE: U44.15 (D3)
- new net PC_INC: U45.19 (D7)
- new net PC_OE: U51.9
- new net PC_WE: U51.6
- new net RAM_OE: U45.18 (D6)
- new net RAM_WE: U45.17 (D5)
- new net STEP0: U44.10 (A0), U45.10 (A0), U46.10 (A0)
- new net STEP1: U44.9 (A1), U45.9 (A1), U46.9 (A1)
- new net STEP2: U44.8 (A2), U45.8 (A2), U46.8 (A2)
- new net VCC: U44.27 (~{WE}), U44.28 (VCC), U45.27 (~{WE}), U45.28 (VCC), U46.27 (~{WE}), U46.28 (VCC), U47.16 (VCC), U48.16 (VCC), U49.16 (VCC), U50.16 (VCC), U51.14 (VDD), U52.14 (VCC), U53.14 (VCC), U54.14 (VCC)
- no-connect marks 0 -> 9
Other:
- note added: "ROM 0-7"
- note added: "ROM 16-23"
- note added: "ROM 8-15"
