File: circuit/ram.kicad_sch (KiCad schematic)
At the start: 29 parts

Commit message: update
Parts:
- removed U? (x6): 74LS08, symbol 74xx:74LS08
- added U29, U57, U58: 74LS08, symbol 74xx:74LS08
- added U34, U41: 74HC273, symbol 74xx:74HC273
- added U55, U56: 74HCT541, symbol 74xx:74HCT541
- gave numbers to parts that had none: 17
Connections:
- net A0: now also U55.18 (Y0)
- net A1: now also U55.17 (Y1)
- net A10: now also U56.16 (Y2)
- net A11: now also U56.15 (Y3)
- net A12: now also U56.14 (Y4)
- net A13: now also U56.13 (Y5)
- net A14: now also U56.12 (Y6)
- net A15: now also U56.11 (Y7)
- net A2: now also U55.16 (Y2)
- net A3: now also U55.15 (Y3)
- net A4: now also U55.14 (Y4)
- net A5: now also U55.13 (Y5)
- net A6: now also U55.12 (Y6)
- net A7: now also U55.11 (Y7)
- net A8: now also U56.18 (Y0)
- net A9: now also U56.17 (Y1)
- net CLK: now also U29.10, U29.13, U29.2, U29.5, U57.10, U57.13, U57.2, U57.5
- net GND: now also U34.10 (GND), U41.10 (GND), U55.10 (GND), U55.19 (G2), U56.10 (GND), U56.19 (G2)
- net IR_WE: now also U57.1, U57.4
- net MAR_WE: now also U29.1, U29.4
- net MD0: now also U34.3 (D0)
- net MD1: now also U34.4 (D1)
- net MD10: now also U41.7 (D2)
- net MD11: now also U41.8 (D3)
- net MD12: now also U41.13 (D4)
- net MD13: now also U41.14 (D5)
- net MD14: now also U41.17 (D6)
- net MD15: now also U41.18 (D7)
- net MD2: now also U34.7 (D2)
- net MD3: now also U34.8 (D3)
- net MD4: now also U34.13 (D4)
- net MD5: now also U34.14 (D5)
- net MD6: now also U34.17 (D6)
- net MD7: now also U34.18 (D7)
- net MD8: now also U41.3 (D0)
- net MD9: now also U41.4 (D1)
- net MDR_WE: now also U29.12, U29.9, U57.12, U57.9
- net VCC: now also U34.1 (~{Mr}), U34.20 (VCC), U41.1 (~{Mr}), U41.20 (VCC), U55.20 (VCC), U56.20 (VCC)
- net at U35.11 (Cp): now also U57.8
- net at U31.11 (Cp): now also U29.6
- net at U43.11 (Cp): now also U57.6
- net I12: now reaches U43.12 (Q4)
- net I13: now reaches U43.15 (Q5)
- net I14: now reaches U43.16 (Q6)
- net I15: now reaches U43.19 (Q7)
- net I8: now reaches U43.2 (Q0)
- net I9: now reaches U43.5 (Q1)
- net I10: now reaches U43.6 (Q2)
- net I11: now reaches U43.9 (Q3)
- net at U42.11 (Cp): now also U57.3
- net at U30.11 (Cp): now also U29.3
- net I4: now reaches U42.12 (Q4)
- net I5: now reaches U42.15 (Q5)
- net I6: now reaches U42.16 (Q6)
- net I7: now reaches U42.19 (Q7)
- net I0: now reaches U42.2 (Q0)
- net I1: now reaches U42.5 (Q1)
- net I2: now reaches U42.6 (Q2)
- net I3: now reaches U42.9 (Q3)
- net at U36.11 (Cp): now also U57.11
- new net: U29.11, U41.11 (Cp)
- new net: U41.12 (Q4), U56.6 (A4)
- new net: U41.15 (Q5), U56.7 (A5)
- new net: U41.16 (Q6), U56.8 (A6)
- new net: U41.19 (Q7), U56.9 (A7)
- new net: U41.2 (Q0), U56.2 (A0)
- new net: U41.5 (Q1), U56.3 (A1)
- new net: U41.6 (Q2), U56.4 (A2)
- new net: U41.9 (Q3), U56.5 (A3)
- new net: U34.2 (Q0), U55.2 (A0)
- new net: U34.5 (Q1), U55.3 (A1)
- new net: U34.6 (Q2), U55.4 (A2)
- new net: U34.9 (Q3), U55.5 (A3)
- new net: U34.12 (Q4), U55.6 (A4)
- new net: U34.15 (Q5), U55.7 (A5)
- new net: U34.16 (Q6), U55.8 (A6)
- new net: U34.19 (Q7), U55.9 (A7)
- new net: U29.8, U34.11 (Cp)
- new net PC_OE: U55.1 (G1), U56.1 (G1)
Other:
- note added: "PC Register"
- moved on the sheet: U24, U25, U26, U27, U28A, U28B, U28C, U28D, U28E, U28F, U28G, U30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
